File: kicad/a500-sd-plus-controller/a500-sd-plus-controller.kicad_pcb (KiCad board)
At the start: 4 copper layers, 84 x 51 mm, 83 parts, among them J1 JTAG, J2 Conn_01x02, J3 Micro_SD_Card_Det2, J4 Micro_SD_Card_Det2, J5 RJ45, K1 DIP_socket_40pins, Q1 AO3400A, U1 5M160ZE64, U10 ENC28J60x-SS, U2 SN74LVC4245A, U3 SN74LVC4245A, U4 CSG8520_CIA, U5 RT9013-18, U6 RT9013-33, U7 RT9013-33, U8 RT9013-33, U9 SRV05-4, Y1 16MHz, Y2 25.0MHz

Commit message: PCB done, this version has been sent to fabrication
Parts:
- added R27: 68K, Resistor_SMD:R_0603_1608Metric, F.Cu at (168.4, 103.1)
- C23, C26: value 22p -> 22pF
- R1, R11, R2, R3, R4, R5, R6, R7, R8: value 47E -> 100R
- R10, R19, R21: value 100E -> 470R
- R12, R13, R14, R15, R16, R9: value 100E -> 100R
- R20: value 0E -> 0R
- R22: value 2K32 -> 2K4
- R23, R24, R25, R26: value 49K9 -> 49R9
- U10: value ENC28J60x-SS -> ENC28J60
- moved C21 4.03 mm to (173.5, 108.5), turned to 0 degrees
- moved C18 1.53 mm to (173.5, 102.1), turned to 0 degrees
- moved U8 1.45 mm to (173.5, 105.3), turned to -90 degrees
- moved U9 1.27 mm to (172.8, 112.8)
- moved R22 1.14 mm to (169.9, 103.1)
- moved REF** 0.18 mm to (172.5, 92.5)
- moved REF** 0.08 mm to (121.0, 112.4)
Routing:
- net /Micro-SD/+3V3_SD2: track 33.2 -> 24.4 mm, vias 2 -> 3
- net VCC: track 193.9 -> 200.7 mm
- net Net-(J4-DAT0): track 31.8 -> 30.6 mm
- net Net-(U10-RBIAS): track 2.46 -> 3.61 mm
- net GND: track 119.1 -> 119.4 mm, vias 49 -> 50
