File: kicad/a500-sd-plus-controller/a500-sd-plus-controller.kicad_pcb (KiCad board)
At the start: 4 copper layers, 84 x 51 mm, 84 parts, among them J1 JTAG, J2 Conn_01x02, J3 Micro_SD_Card_Det2, J4 Micro_SD_Card_Det2, J5 RJ45, K1 DIP_socket_40pins, Q1 AO3400A, U1 5M160ZE64, U10 ENC28J60, U2 SN74LVC4245A, U3 SN74LVC4245A, U4 CSG8520_CIA, U5 RT9013-18, U6 RT9013-33, U7 RT9013-33, U8 RT9013-33, U9 SRV05-4, Y1 16MHz, Y2 25.0MHz

Commit message: Fill in C13 sourcing, flag U4 as not-populated, thicken thin silkscreen
Three small fixes found while preparing a fabrication package.

C13 (100uF/16V) was the only part in the schematic with neither an MPN nor
an LCSC part number, so any assembly quote stalls on it. Added AISHI
EH71CM101E07OT / C112487: 100uF 16V, 6.3mm diameter, 2.5mm lead pitch,
7mm seated height. That fits CP_Radial_D8.0mm_P2.50mm with margin and is
the shortest 16V part in that pitch, which matters given how little room
there is above the board.

U4 is the 8520 CIA harvested from the A500 motherboard -- its pads are
where the turned pin headers go, and no assembly house should ever place
it. Marked DNP in the schematic and on the footprint, so it now drops out
of position files automatically while still appearing in BOM exports with
a DNP flag. Left "exclude from BOM" off deliberately: hiding it entirely
loses the information that the part exists.

Two silkscreen texts, JTAG (0.10mm) and HDD/LED (0.125mm), were below the
0.15mm minimum stroke width most fabs quote, PCBWay included, so they risk
printing faintly. Bumped both to 0.15mm. Text size is unchanged, and DRC
is unaffected: still 0 unconnected, 0 footprint errors, and the same 12
pre-existing courtyard overlaps under U4.
Changed lines of the file:
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@@
 		(sheetname "/Mainboard interface/")
 		(sheetfile "mainboard_riser.kicad_sch")
-		(attr through_hole)
+		(attr through_hole dnp)
 		(fp_line
 			(start 1.16 49.59)
@@
 			(font
 				(size 1 1)
-				(thickness 0.1)
+				(thickness 0.15)
 			)
 			(justify left bottom)
@@
 			(font
 				(size 1 1)
-				(thickness 0.125)
+				(thickness 0.15)
 			)
 			(justify left bottom)
