File: kicad/a500-sd-plus-controller/mainboard_riser.kicad_sch (KiCad schematic)
At the start: 2 parts, among them K1 DIP_socket_40pins, U4 CSG8520_CIA

Commit message: Fill in C13 sourcing, flag U4 as not-populated, thicken thin silkscreen
Three small fixes found while preparing a fabrication package.

C13 (100uF/16V) was the only part in the schematic with neither an MPN nor
an LCSC part number, so any assembly quote stalls on it. Added AISHI
EH71CM101E07OT / C112487: 100uF 16V, 6.3mm diameter, 2.5mm lead pitch,
7mm seated height. That fits CP_Radial_D8.0mm_P2.50mm with margin and is
the shortest 16V part in that pitch, which matters given how little room
there is above the board.

U4 is the 8520 CIA harvested from the A500 motherboard -- its pads are
where the turned pin headers go, and no assembly house should ever place
it. Marked DNP in the schematic and on the footprint, so it now drops out
of position files automatically while still appearing in BOM exports with
a DNP flag. Left "exclude from BOM" off deliberately: hiding it entirely
loses the information that the part exists.

Two silkscreen texts, JTAG (0.10mm) and HDD/LED (0.125mm), were below the
0.15mm minimum stroke width most fabs quote, PCBWay included, so they risk
printing faintly. Bumped both to 0.15mm. Text size is unchanged, and DRC
is unaffected: still 0 unconnected, 0 footprint errors, and the same 12
pre-existing courtyard overlaps under U4.
Parts:
- U4: now not fitted
Changed lines of the file:
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@@
 		(in_bom yes)
 		(on_board yes)
-		(dnp no)
+		(dnp yes)
 		(fields_autoplaced yes)
 		(property "Reference" "U4"
